File: ergogen-out/pcbs/banana_split.kicad_pcb (KiCad board)
At the start: 2 copper layers, 299.9 x 109 mm, 86 parts

Commit message: net names for left
Parts:
- added B1: , E73:SW_TACT_ALPS_SKQGABE010, F.Cu at (88.1, 98.7)
- added B2: , E73:SW_TACT_ALPS_SKQGABE010, F.Cu at (351.0, 98.7)
Connections:
- D1 pad 1: (no net) -> P031
- D10 pad 1: (no net) -> P031
- D11 pad 1: (no net) -> P029
- D12 pad 1: (no net) -> P002
- D13 pad 1: (no net) -> P031
- D14 pad 1: (no net) -> P029
- D15 pad 1: (no net) -> P002
- D19 pad 1: (no net) -> P115
- D2 pad 1: (no net) -> P029
- D20 pad 1: (no net) -> P115
- D21 pad 1: (no net) -> P031
- D22 pad 1: (no net) -> P029
- D23 pad 1: (no net) -> P002
- D24 pad 1: (no net) -> P031
- D25 pad 1: (no net) -> P029
- D26 pad 1: (no net) -> P002
- D27 pad 1: (no net) -> P031
- D28 pad 1: (no net) -> P029
- D29 pad 1: (no net) -> P002
- D3 pad 1: (no net) -> P002
- D30 pad 1: (no net) -> P031
- D31 pad 1: (no net) -> P029
- D32 pad 1: (no net) -> P002
- D33 pad 1: (no net) -> P031
- D34 pad 1: (no net) -> P029
- D35 pad 1: (no net) -> P002
- D39 pad 1: (no net) -> P115
- D4 pad 1: (no net) -> P031
- D40 pad 1: (no net) -> P115
- D5 pad 1: (no net) -> P029
- D6 pad 1: (no net) -> P002
- D7 pad 1: (no net) -> P031
- D8 pad 1: (no net) -> P029
- D9 pad 1: (no net) -> P002
- S1 pad 1: (no net) -> P022
- S10 pad 1: (no net) -> P011
- S11 pad 1: (no net) -> P011
- S12 pad 1: (no net) -> P011
- S13 pad 1: (no net) -> P104
- S14 pad 1: (no net) -> P104
- S15 pad 1: (no net) -> P104
- S16 pad 1: (no net) -> P022
- S17 pad 1: (no net) -> P024
- S18 pad 1: (no net) -> P100
- S19 pad 1: (no net) -> P011
- S2 pad 1: (no net) -> P022
- S20 pad 1: (no net) -> P104
- S21 pad 1: (no net) -> P022
- S22 pad 1: (no net) -> P022
- S23 pad 1: (no net) -> P022
- S24 pad 1: (no net) -> P024
- S25 pad 1: (no net) -> P024
- S26 pad 1: (no net) -> P024
- S27 pad 1: (no net) -> P100
- S28 pad 1: (no net) -> P100
- S29 pad 1: (no net) -> P100
- S3 pad 1: (no net) -> P022
- S30 pad 1: (no net) -> P011
- S31 pad 1: (no net) -> P011
- S32 pad 1: (no net) -> P011
- S33 pad 1: (no net) -> P104
- S34 pad 1: (no net) -> P104
- S35 pad 1: (no net) -> P104
- S36 pad 1: (no net) -> P022
- S37 pad 1: (no net) -> P024
- S38 pad 1: (no net) -> P100
- S39 pad 1: (no net) -> P011
- S4 pad 1: (no net) -> P024
- S40 pad 1: (no net) -> P104
- S5 pad 1: (no net) -> P024
- S6 pad 1: (no net) -> P024
- S7 pad 1: (no net) -> P100
- S8 pad 1: (no net) -> P100
- S9 pad 1: (no net) -> P100

Commit message: fix net names
Connections:
- D21 pad 1: P031 -> RP031
- D22 pad 1: P029 -> RP029
- D23 pad 1: P002 -> RP002
- D24 pad 1: P031 -> RP031
- D25 pad 1: P029 -> RP029
- D26 pad 1: P002 -> RP002
- D27 pad 1: P031 -> RP031
- D28 pad 1: P029 -> RP029
- D29 pad 1: P002 -> RP002
- D30 pad 1: P031 -> RP031
- D31 pad 1: P029 -> RP029
- D32 pad 1: P002 -> RP002
- D33 pad 1: P031 -> RP031
- D34 pad 1: P029 -> RP029
- D35 pad 1: P002 -> RP002
- D39 pad 1: P115 -> RP115
- D40 pad 1: P115 -> RP115
- S21 pad 1: P022 -> RP022
- S22 pad 1: P022 -> RP022
- S23 pad 1: P022 -> RP022
- S24 pad 1: P024 -> RP024
- S25 pad 1: P024 -> RP024
- S26 pad 1: P024 -> RP024
- S27 pad 1: P100 -> RP100
- S28 pad 1: P100 -> RP100
- S29 pad 1: P100 -> RP100
- S30 pad 1: P011 -> RP011
- S31 pad 1: P011 -> RP011
- S32 pad 1: P011 -> RP011
- S33 pad 1: P104 -> RP104
- S34 pad 1: P104 -> RP104
- S35 pad 1: P104 -> RP104
- S36 pad 1: P022 -> RP022
- S37 pad 1: P024 -> RP024
- S38 pad 1: P100 -> RP100
- S39 pad 1: P011 -> RP011
- S40 pad 1: P104 -> RP104

Commit message: remove reversibility
Connections:
- JST1 pad 1: RAW -> GND
- JST1 pad 2: GND -> RAW
- JST2 pad 1: RRAW -> RGND
- JST2 pad 2: RGND -> RRAW
Routing:
- net JST1_1: track 3.60 -> 0.00 mm
- net JST2_2: track 3.60 -> 0.00 mm
- net JST2_1: track 3.60 -> 0.00 mm
- net JST1_2: track 3.60 -> 0.00 mm

Commit message: pcb routed
Connections:
- D16 pad 1: (no net) -> P115
- D17 pad 1: (no net) -> P115
- D18 pad 1: (no net) -> P115
- D36 pad 1: (no net) -> RP115
- D37 pad 1: (no net) -> RP115
- D38 pad 1: (no net) -> RP115
Changed lines of the file:
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@@
         (fp_line (start -0.35 0) (end -0.35 -0.55) (layer B.SilkS) (width 0.1))
         (fp_line (start -0.75 0) (end -0.35 0) (layer B.SilkS) (width 0.1))
-        (pad 1 smd rect (at -1.65 0 -10) (size 0.9 1.2) (layers F.Cu F.Paste F.Mask) (net 0 ""))
+        (pad 1 smd rect (at -1.65 0 -10) (size 0.9 1.2) (layers F.Cu F.Paste F.Mask) (net 54 "P115"))
         (pad 2 smd rect (at 1.65 0 -10) (size 0.9 1.2) (layers B.Cu B.Paste B.Mask) (net 21 "in_thumb"))
-        (pad 1 smd rect (at -1.65 0 -10) (size 0.9 1.2) (layers B.Cu B.Paste B.Mask) (net 0 ""))
+        (pad 1 smd rect (at -1.65 0 -10) (size 0.9 1.2) (layers B.Cu B.Paste B.Mask) (net 54 "P115"))
         (pad 2 smd rect (at 1.65 0 -10) (size 0.9 1.2) (layers F.Cu F.Paste F.Mask) (net 21 "in_thumb"))
-        (pad 1 thru_hole rect (at -3.81 0 -10) (size 1.778 1.778) (drill 0.9906) (layers *.Cu *.Mask) (net 0 ""))
+        (pad 1 thru_hole rect (at -3.81 0 -10) (size 1.778 1.778) (drill 0.9906) (layers *.Cu *.Mask) (net 54 "P115"))
         (pad 2 thru_hole circle (at 3.81 0 -10) (size 1.905 1.905) (drill 0.9906) (layers *.Cu *.Mask) (net 21 "in_thumb"))
     )
@@
         (fp_line (start -0.35 0) (end -0.35 -0.55) (layer B.SilkS) (width 0.1))
         (fp_line (start -0.75 0) (end -0.35 0) (layer B.SilkS) (width 0.1))
-        (pad 1 smd rect (at -1.65 0 -30) (size 0.9 1.2) (layers F.Cu F.Paste F.Mask) (net 0 ""))
+        (pad 1 smd rect (at -1.65 0 -30) (size 0.9 1.2) (layers F.Cu F.Paste F.Mask) (net 54 "P115"))
         (pad 2 smd rect (at 1.65 0 -30) (size 0.9 1.2) (layers B.Cu B.Paste B.Mask) (net 22 "home_thumb"))
-        (pad 1 smd rect (at -1.65 0 -30) (size 0.9 1.2) (layers B.Cu B.Paste B.Mask) (net 0 ""))
+        (pad 1 smd rect (at -1.65 0 -30) (size 0.9 1.2) (layers B.Cu B.Paste B.Mask) (net 54 "P115"))
         (pad 2 smd rect (at 1.65 0 -30) (size 0.9 1.2) (layers F.Cu F.Paste F.Mask) (net 22 "home_thumb"))
-        (pad 1 thru_hole rect (at -3.81 0 -30) (size 1.778 1.778) (drill 0.9906) (layers *.Cu *.Mask) (net 0 ""))
+        (pad 1 thru_hole rect (at -3.81 0 -30) (size 1.778 1.778) (drill 0.9906) (layers *.Cu *.Mask) (net 54 "P115"))
         (pad 2 thru_hole circle (at 3.81 0 -30) (size 1.905 1.905) (drill 0.9906) (layers *.Cu *.Mask) (net 22 "home_thumb"))
     )
@@
         (fp_line (start -0.35 0) (end -0.35 -0.55) (layer B.SilkS) (width 0.1))
         (fp_line (start -0.75 0) (end -0.35 0) (layer B.SilkS) (width 0.1))
-        (pad 1 smd rect (at -1.65 0 -53) (size 0.9 1.2) (layers F.Cu F.Paste F.Mask) (net 0 ""))
+        (pad 1 smd rect (at -1.65 0 -53) (size 0.9 1.2) (layers F.Cu F.Paste F.Mask) (net 54 "P115"))
         (pad 2 smd rect (at 1.65 0 -53) (size 0.9 1.2) (layers B.Cu B.Paste B.Mask) (net 23 "out_thumb"))
-        (pad 1 smd rect (at -1.65 0 -53) (size 0.9 1.2) (layers B.Cu B.Paste B.Mask) (net 0 ""))
+        (pad 1 smd rect (at -1.65 0 -53) (size 0.9 1.2) (layers B.Cu B.Paste B.Mask) (net 54 "P115"))
         (pad 2 smd rect (at 1.65 0 -53) (size 0.9 1.2) (layers F.Cu F.Paste F.Mask) (net 23 "out_thumb"))
-        (pad 1 thru_hole rect (at -3.81 0 -53) (size 1.778 1.778) (drill 0.9906) (layers *.Cu *.Mask) (net 0 ""))
+        (pad 1 thru_hole rect (at -3.81 0 -53) (size 1.778 1.778) (drill 0.9906) (layers *.Cu *.Mask) (net 54 "P115"))
         (pad 2 thru_hole circle (at 3.81 0 -53) (size 1.905 1.905) (drill 0.9906) (layers *.Cu *.Mask) (net 23 "out_thumb"))
     )
@@
         (fp_line (start -0.35 0) (end -0.35 -0.55) (layer B.SilkS) (width 0.1))
         (fp_line (start -0.75 0) (end -0.35 0) (layer B.SilkS) (width 0.1))
-        (pad 1 smd rect (at -1.65 0 10) (size 0.9 1.2) (layers F.Cu F.Paste F.Mask) (net 0 ""))
+        (pad 1 smd rect (at -1.65 0 10) (size 0.9 1.2) (layers F.Cu F.Paste F.Mask) (net 58 "RP115"))
         (pad 2 smd rect (at 1.65 0 10) (size 0.9 1.2) (layers B.Cu B.Paste B.Mask) (net 46 "mirror_in_thumb"))
-        (pad 1 smd rect (at -1.65 0 10) (size 0.9 1.2) (layers B.Cu B.Paste B.Mask) (net 0 ""))
+        (pad 1 smd rect (at -1.65 0 10) (size 0.9 1.2) (layers B.Cu B.Paste B.Mask) (net 58 "RP115"))
         (pad 2 smd rect (at 1.65 0 10) (size 0.9 1.2) (layers F.Cu F.Paste F.Mask) (net 46 "mirror_in_thumb"))
-        (pad 1 thru_hole rect (at -3.81 0 10) (size 1.778 1.778) (drill 0.9906) (layers *.Cu *.Mask) (net 0 ""))
+        (pad 1 thru_hole rect (at -3.81 0 10) (size 1.778 1.778) (drill 0.9906) (layers *.Cu *.Mask) (net 58 "RP115"))
         (pad 2 thru_hole circle (at 3.81 0 10) (size 1.905 1.905) (drill 0.9906) (layers *.Cu *.Mask) (net 46 "mirror_in_thumb"))
     )
@@
         (fp_line (start -0.35 0) (end -0.35 -0.55) (layer B.SilkS) (width 0.1))
         (fp_line (start -0.75 0) (end -0.35 0) (layer B.SilkS) (width 0.1))
-        (pad 1 smd rect (at -1.65 0 30) (size 0.9 1.2) (layers F.Cu F.Paste F.Mask) (net 0 ""))
+        (pad 1 smd rect (at -1.65 0 30) (size 0.9 1.2) (layers F.Cu F.Paste F.Mask) (net 58 "RP115"))
         (pad 2 smd rect (at 1.65 0 30) (size 0.9 1.2) (layers B.Cu B.Paste B.Mask) (net 47 "mirror_home_thumb"))
-        (pad 1 smd rect (at -1.65 0 30) (size 0.9 1.2) (layers B.Cu B.Paste B.Mask) (net 0 ""))
+        (pad 1 smd rect (at -1.65 0 30) (size 0.9 1.2) (layers B.Cu B.Paste B.Mask) (net 58 "RP115"))
         (pad 2 smd rect (at 1.65 0 30) (size 0.9 1.2) (layers F.Cu F.Paste F.Mask) (net 47 "mirror_home_thumb"))
-        (pad 1 thru_hole rect (at -3.81 0 30) (size 1.778 1.778) (drill 0.9906) (layers *.Cu *.Mask) (net 0 ""))
+        (pad 1 thru_hole rect (at -3.81 0 30) (size 1.778 1.778) (drill 0.9906) (layers *.Cu *.Mask) (net 58 "RP115"))
         (pad 2 thru_hole circle (at 3.81 0 30) (size 1.905 1.905) (drill 0.9906) (layers *.Cu *.Mask) (net 47 "mirror_home_thumb"))
     )
@@
         (fp_line (start -0.35 0) (end -0.35 -0.55) (layer B.SilkS) (width 0.1))
         (fp_line (start -0.75 0) (end -0.35 0) (layer B.SilkS) (width 0.1))
-        (pad 1 smd rect (at -1.65 0 53) (size 0.9 1.2) (layers F.Cu F.Paste F.Mask) (net 0 ""))
+        (pad 1 smd rect (at -1.65 0 53) (size 0.9 1.2) (layers F.Cu F.Paste F.Mask) (net 58 "RP115"))
         (pad 2 smd rect (at 1.65 0 53) (size 0.9 1.2) (layers B.Cu B.Paste B.Mask) (net 48 "mirror_out_thumb"))
-        (pad 1 smd rect (at -1.65 0 53) (size 0.9 1.2) (layers B.Cu B.Paste B.Mask) (net 0 ""))
+        (pad 1 smd rect (at -1.65 0 53) (size 0.9 1.2) (layers B.Cu B.Paste B.Mask) (net 58 "RP115"))
         (pad 2 smd rect (at 1.65 0 53) (size 0.9 1.2) (layers F.Cu F.Paste F.Mask) (net 48 "mirror_out_thumb"))
-        (pad 1 thru_hole rect (at -3.81 0 53) (size 1.778 1.778) (drill 0.9906) (layers *.Cu *.Mask) (net 0 ""))
+        (pad 1 thru_hole rect (at -3.81 0 53) (size 1.778 1.778) (drill 0.9906) (layers *.Cu *.Mask) (net 58 "RP115"))
         (pad 2 thru_hole circle (at 3.81 0 53) (size 1.905 1.905) (drill 0.9906) (layers *.Cu *.Mask) (net 48 "mirror_out_thumb"))
     )
