File: ergogen-out/pcbs/routed_banana_split.kicad_pcb (KiCad board)
At the start: 2 copper layers, 299.9 x 109 mm, 88 parts

Commit message: render 1
Routing:
- net RP022: track 252.5 -> 256.7 mm
- net RP006: track 41.9 -> 45.0 mm
- net P022: track 249.4 -> 246.9 mm
- net RGND: track 240.2 -> 239.2 mm
Other:
- outline, holes or cut-outs redrawn
- board text added: "Banana Split"
